Commit message: proper orientation of urdf

File: docs/module1/lab1_building_robot/code/rosjet/jet_description/urdf/jet.xacro (robot description, xacro)
@@ -6,8 +6,10 @@
   <xacro:include filename="$(find jet_description)/urdf/materials.xacro"/>
   <link name="base_link">
-    <visual>
-      <origin rpy="0 0 0" xyz="0 0 0"/>
-      <geometry>
-        <box size=".25 .35 .05"/>
+  </link>
+  <link name="body_link">
+    <visual>
+      <origin rpy="0 0 0" xyz="0 0 0"/>
+      <geometry>
+        <box size=".35 .25 .05"/>
       </geometry>
       <material name="green">
@@ -18,5 +20,5 @@
       <origin rpy="0 0 0" xyz="0 0 0"/>
       <geometry>
-        <box size=".25 .35 .05"/>
+        <box size=".35 .25 .05"/>
       </geometry>
     </collision>
@@ -28,5 +30,5 @@
   <link name="caster">
     <visual name='caster_visual'>
-      <origin rpy="0 0 0" xyz="0 .15 -.06"/>
+      <origin rpy="0 0 0" xyz="0 0 0"/>
       <geometry>
         <cylinder radius="0.03" length="0.12"/>
@@ -34,5 +36,5 @@
     </visual>
     <collision name='caster_collision'>
-      <origin rpy="0 0 0" xyz="0 .15 -.06"/>
+      <origin rpy="0 0 0" xyz="0 0 0"/>
       <geometry>
         <cylinder radius="0.03" length="0.12"/>
@@ -59,5 +61,5 @@
         <cylinder length="0.03" radius="0.1"/>
       </geometry>
-      <origin rpy="0 1.57075 0" xyz="0 0 0"/>
+      <origin rpy="0 1.57075 1.57075" xyz="0 0 0"/>
       <material name="gray">
         <color rgba=".1 .1 .1 1"/>
@@ -68,5 +70,5 @@
         <cylinder length="0.03" radius="0.1"/>
       </geometry>
-      <origin rpy="0 1.57075 0" xyz="0 0 0"/>
+      <origin rpy="0 1.57075 1.57075" xyz="0 0 0"/>
     </collision>
     <inertial>
@@ -80,5 +82,5 @@
         <cylinder length="0.03" radius="0.1"/>
       </geometry>
-      <origin rpy="0 1.57075 0" xyz="0 0 0"/>
+      <origin rpy="0 1.57075 1.57075" xyz="0 0 0"/>
       <material name="gray">
         <color rgba=".1 .1 .1 1"/>
@@ -89,5 +91,5 @@
         <cylinder length="0.03" radius="0.1"/>
       </geometry>
-      <origin rpy="0 1.57075 0" xyz="0 0 0"/>
+      <origin rpy="0 1.57075 1.57075" xyz="0 0 0"/>
     </collision>
     <inertial>
@@ -119,5 +121,5 @@
   <link name="camera_link">
     <collision>
-      <origin xyz="0 0 0" rpy="0 0 -1.57075"/>
+      <origin xyz="0 0 0" rpy="0 0 0"/>
       <geometry>
         <box size=".05 .02 .05"/>
@@ -125,5 +127,5 @@
     </collision>
     <visual>
-      <origin xyz="0 0 0" rpy="0 0 -1.57075"/>
+      <origin xyz="0 0 0" rpy="0 0 0"/>
       <geometry>
         <box size=".05 .02 .05"/>
@@ -146,8 +148,14 @@
     </inertial>
   </link>
+  <joint name="body_base" type="fixed">
+    <axis xyz="1 0 0"/>
+    <origin xyz="0 0 0"/>
+    <parent link="base_link"/>
+    <child link="body_link"/>
+  </joint>
   <joint name="imu_joint" type="fixed">
     <axis xyz="1 0 0"/>
     <origin xyz="0 0 0"/>
-    <parent link="base_link"/>
+    <parent link="body_link"/>
     <child link="gyro_link"/>
   </joint>
@@ -155,5 +163,5 @@
       <axis xyz="0 1 0" />
       <origin xyz="-.1 -.15 -.05" rpy="0 0 -2.356125"/>
-      <parent link="base_link"/>
+      <parent link="body_link"/>
       <child link="sonar1_link"/>
   </joint>
@@ -161,5 +169,5 @@
       <axis xyz="0 1 0" />
       <origin xyz="0 -.15 -.05" rpy="0 0 -1.57075"/>
-      <parent link="base_link"/>
+      <parent link="body_link"/>
       <child link="sonar2_link"/>
   </joint>
@@ -167,31 +175,31 @@
       <axis xyz="0 1 0" />
       <origin xyz=".1 -.15 -.05" rpy="0 0 -.785375"/>
-      <parent link="base_link"/>
+      <parent link="body_link"/>
       <child link="sonar3_link"/>
   </joint>
   <joint name="camera_joint" type="fixed">
-      <axis xyz="0 1 0" />
-      <origin xyz="0 -.15 .05" rpy="0 0 0"/>
-      <parent link="base_link"/>
+      <axis xyz="1 0 0" />
+      <origin xyz=".15 0 .05" rpy="0 0 0"/>
+      <parent link="body_link"/>
       <child link="camera_link"/>
   </joint>
   <joint name="caster_base_joint" type="fixed">
-    <parent link="base_link"/>
+    <parent link="body_link"/>
     <child link="caster"/>
-    <origin xyz="0 0 0"/>
+    <origin xyz="-.15 0 -.05"/>
     <axis xyz="0 0 1"/>
   </joint>
   <joint name="right_wheel_joint" type="revolute">
-    <parent link="base_link"/>
+    <parent link="body_link"/>
     <child link="right_wheel"/>
-    <origin xyz="0.15 -.05 -.03"/>
-    <axis xyz="1 0 0"/>
+    <origin xyz="0.08 -.15 -.03"/>
+    <axis xyz="0 1 0"/>
     <limit effort="100" velocity="100.0" lower="-5000" upper="5000" />
   </joint>
   <joint name="left_wheel_joint" type="revolute">
-    <parent link="base_link"/>
+    <parent link="body_link"/>
     <child link="left_wheel"/>
-    <origin xyz="-0.15 -.05 -.03"/>
-    <axis xyz="1 0 0"/>
+    <origin xyz="0.08 .15 -.03"/>
+    <axis xyz="0 1 0"/>
     <limit effort="100" velocity="100.0" lower="-5000" upper="5000"/>
   </joint>
